Commit message: minor edits

File: urdf/robot.urdf (robot description, URDF)
Before this commit: robot pioneer3at, 2 links, 1 joints
Links:
- link base_laser: geometry collision box size=0.1 0.1 0.1; visual box size=0.1 0.1 0.1
Joints:
- joint base_laser_joint: origin xyz=0 0 0 rpy=0 0 0 -> xyz=2 0 0 rpy=0 0 0
